File: node/robot.kicad_sch (KiCad schematic)
At the start: 25 parts, among them J1 Conn_01x19_Female, J2 Conn_01x19_Female

Commit message: add node for reference
Parts:
- removed M? (x2): MPMOS, symbol pspice:MPMOS
- removed M? (x2): MNMOS, symbol pspice:MNMOS
- removed M?: Motor_DC, symbol Motor:Motor_DC
- removed R? (x4): 5k, Resistor_THT:R_Axial_DIN0614_L14.3mm_D5.7mm_P15.24mm_Horizontal, symbol Device:R
- removed U? (x2): NSL-32, OptoDevice:Luna_NSL-32, symbol Isolator:NSL-32
- added M10: Motor_DC, symbol Motor:Motor_DC
- added M6, M7: MPMOS, symbol pspice:MPMOS
- added M8, M9: MNMOS, symbol pspice:MNMOS
- added R5, R8: 1k, Resistor_THT:R_Axial_DIN0614_L14.3mm_D5.7mm_P15.24mm_Horizontal, symbol Device:R
- added R6, R7: 47k, Resistor_THT:R_Axial_DIN0614_L14.3mm_D5.7mm_P15.24mm_Horizontal, symbol Device:R
- added U3, U4: NSL-32, OptoDevice:Luna_NSL-32, symbol Isolator:NSL-32
- R1, R4: renamed from R?; value 5k -> 1k
- R2, R3: renamed from R?; value 5k -> 47k
- gave numbers to parts that had none: 7
Connections:
- net 3.3V: now also R5.2, R8.2
- net 6V: now also M6.3 (S), M6.4 (B), M7.3 (S), M7.4 (B), R6.2, R7.2
- net GND: now also M8.3 (S), M8.4 (B), M9.3 (S), M9.4 (B), U3.3 (R), U4.3 (R)
- net M11: now also U3.2 (K)
- net M12: now also U4.2 (K)
- new net: M7.2 (G), M9.2 (G), R7.1, U4.4 (R)
- new net: M10.1 (+), M6.1 (D), M8.1 (D)
- new net: M10.2 (-), M7.1 (D), M9.1 (D)
- new net: R8.1, U4.1 (A)
- new net: R5.1, U3.1 (A)
- new net: M6.2 (G), M8.2 (G), R6.1, U3.4 (R)
Other:
- moved on the sheet: J1, J2, J?
