File: kicad/robot_pcb.kicad_sch (KiCad schematic)
At the start: 27 parts, among them J1 Conn_01x19_Female, J2 Conn_01x19_Female, J3 esp32 cam, J4 motor1, J5 motor2, J6 motor pwr, J7 esp32 pwr, Q1 Q_PMOS_GDS, Q2 Q_NMOS_GDS, Q3 Q_PMOS_GDS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

Commit message: pcb rev 2
Parts:
- removed Q1, Q3, Q5, Q7: Q_PMOS_GDS, Downloads:SOIC127P490X600X175-8N, symbol Device:Q_PMOS_GDS
- removed Q2, Q4, Q6, Q8: Q_NMOS_GDS, Downloads:SOIC127P490X600X175-8N, symbol Device:Q_NMOS_GDS
- added Q1, Q3, Q5, Q7: AO3401A, digikey-footprints:SOT-23-3, symbol dk_Transistors-FETs-MOSFETs-Single:AO3401A
- added Q2, Q4, Q6, Q8: IRLML6344TRPBF, digikey-footprints:SOT-23-3, symbol dk_Transistors-FETs-MOSFETs-Single:IRLML6344TRPBF
- R1, R2, R3, R4, R5, R6, R7, R8: footprint Resistor_SMD:R_0201_0603Metric_Pad0.64x0.40mm_HandSolder -> Resistor_SMD:R_0805_2012Metric_Pad1.20x1.40mm_HandSolder
Connections:
- net Gate1: now also Q1.1 (G), Q2.1 (G)
- net Gate2: now also Q3.1 (G), Q4.1 (G)
- net Gate3: now also Q5.1 (G), Q6.1 (G)
- net Gate4: now also Q7.1 (G), Q8.1 (G)
- net MGND: now also Q2.2 (S), Q4.2 (S), Q6.2 (S), Q8.2 (S)
- net MO1: now also Q1.3 (D), Q2.3 (D)
- net MO2: now also Q3.3 (D), Q4.3 (D)
- net MO3: now also Q5.3 (D), Q6.3 (D)
- net MO4: now also Q7.3 (D), Q8.3 (D)
- net Vm: now also Q1.2 (S), Q3.2 (S), Q5.2 (S), Q7.2 (S)
Other:
- note added: "December 12, 2022"
- note removed: "November 25, 2022"
